File: sensornode/sensornode_esp32/esp32_sensornode/esp32_sensornode.kicad_pcb (KiCad board)
At the start: 2 copper layers, 70 x 33 mm, 38 parts, among them J1 Conn_01x06_Female, J2 Conn_01x07_Male, J3 Micro_SD_Card, J4 USB_B_Mini, J5 Conn_01x02_Male, J6 Conn_02x03_Odd_Even, J7 Conn_02x03_Odd_Even, Q1 NDS3332P, Q2 NDS3332P, Q3 NDS3332P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

Commit message: create files for ordering
Changed lines of the file:
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@@
       (outputformat 1)
       (mirror false)
-      (drillshape 1)
+      (drillshape 0)
       (scaleselection 1)
-      (outputdirectory ""))
+      (outputdirectory "position"))
   )
   (net 0 "")
@@
     (tags capacitor)
     (attr smd)
-    (fp_text reference C5 (at 0 -1.43) (layer F.SilkS)
+    (fp_text reference C5 (at -2.2606 0.0127) (layer F.SilkS)
       (effects (font (size 1 1) (thickness 0.15)))
     )
@@
   (module logo:diamond (layer F.Cu)
     (at 109.6519 54.5225)
+    (attr smd)
     (fp_text reference G*** (at 0 0) (layer F.SilkS) hide
       (effects (font (size 1.524 1.524) (thickness 0.3)))
@@
   (module progcode-resources:pc3 (layer F.Cu)
     (at 111.6839 49.1123)
+    (attr smd)
     (fp_text reference G*** (at 0 0) (layer F.SilkS) hide
       (effects (font (size 1.524 1.524) (thickness 0.3)))
@@
     (tags resistor)
     (attr smd)
-    (fp_text reference R1 (at 0.9398 -1.3843) (layer F.SilkS)
+    (fp_text reference R1 (at 0.6731 -1.4351) (layer F.SilkS)
       (effects (font (size 1 1) (thickness 0.15)))
     )
@@
     (tags SOT-23)
     (attr smd)
-    (fp_text reference U6 (at -0.1905 2.4638 90) (layer F.SilkS)
+    (fp_text reference U6 (at 0.127 2.7432 180) (layer F.SilkS)
       (effects (font (size 1 1) (thickness 0.15)))
     )
