File: sensornode/sensornode_esp32/esp32_sensornode.sch (KiCad schematic (older format))
At the start: 35 parts, among them J1 Conn_01x06_Female, J2 Conn_01x07_Male, J3 Micro_SD_Card, J4 USB_B_Mini, J5 Conn_01x02_Male, J6 Conn_02x03_Odd_Even, J7 Conn_02x03_Odd_Even, Q1 NDS3332P, Q2 NDS3332P, Q3 NDS3332P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

Commit message: add lcsc part numbers
Parts:
- removed U6: TPS3831, Package_SON:Texas_X2SON-4_1x1mm_P0.65mm, symbol Power_Supervisor:TPS3831
- added U6: TPS3839DBZ, Package_TO_SOT_SMD:SOT-23, symbol Power_Supervisor:TPS3839DBZ
- C1, C3, C4: value 2.2u -> 2.2u 10v; LCSC (none) -> C167329
- C2, C5: value 10u -> 10u 10v; LCSC (none) -> C195004
- J1: LCSC (none) -> C225481
- Q1, Q2, Q3: value NDS3332P -> NDS332P; LCSC (none) -> C258217
- Q4: LCSC (none) -> C96379
- Q5: LCSC (none) -> C151009
- R1, R11, R2: LCSC (none) -> C427267
- R10, R12, R3, R4, R7, R8, R9: LCSC (none) -> C191318
- R5: value R -> 1.18k; LCSC (none) -> C402894
- R6: value R -> 1.13k; LCSC (none) -> C308182
- U1: LCSC (none) -> C95209
- U2: LCSC (none) -> C431940
- U3: LCSC (none) -> C15464
- U4: LCSC (none) -> C108996
- U5: LCSC (none) -> C126019
Connections:
- net labels removed: ~RESET
- wire segments 209 -> 207
Changed lines of the file:
@@
 F 2 "Package_LGA:Bosch_LGA-8_2.5x2.5mm_P0.65mm_ClockwisePinNumbering" H 10325 2475 50  0001 C CNN
 F 3 "https://ae-bst.resource.bosch.com/media/_tech/media/datasheets/BST-BME280-DS002.pdf" H 8825 2725 50  0001 C CNN
+F 4 "C431940" H 8825 2925 50  0001 C CNN "LCSC"
 	1    8825 2925
 	1    0    0    -1
@@
 F 2 "Connector_PinHeader_2.54mm:PinHeader_1x06_P2.54mm_Vertical" H 1750 3950 50  0001 C CNN
 F 3 "~" H 1750 3950 50  0001 C CNN
+F 4 "C225481" H 1750 3950 50  0001 C CNN "LCSC"
 	1    1750 3950
 	1    0    0    -1
@@
 $EndComp
 Text Label 1350 4150 0    50   ~ 0
-~RESET
+EN
 Text Label 1350 4050 0    50   ~ 0
 IO0
@@
 F 2 "RF_Module:ESP32-WROOM-32" H 3700 4550 50  0001 C CNN
 F 3 "https://www.espressif.com/sites/default/files/documentation/esp32-wroom-32_datasheet_en.pdf" H 3400 6100 50  0001 C CNN
+F 4 "C95209" H 3700 6050 50  0001 C CNN "LCSC"
 	1    3700 6050
 	1    0    0    -1
@@
 F 2 "Package_DFN_QFN:QFN-16-1EP_3x3mm_P0.5mm_EP1.7x1.7mm_ThermalVias" H 2400 1475 50  0001 L CNN
 F 3 "http://www.ti.com/lit/ds/symlink/bq24075.pdf" H 2350 2225 50  0001 C CNN
+F 4 "C15464" H 2150 2025 50  0001 C CNN "LCSC"
 	1    2150 2025
 	1    0    0    -1
@@
 F 2 "Package_TO_SOT_SMD:SOT-223-3_TabPin2" H 3800 1575 50  0001 C CNN
 F 3 "http://www.ti.com/lit/ds/symlink/lm1117.pdf" H 3800 1575 50  0001 C CNN
+F 4 "C126019" H 3800 1575 50  0001 C CNN "LCSC"
 	1    3800 1575
 	1    0    0    -1
@@
 P 2500 1150
 F 0 "C1" V 2248 1150 50  0000 C CNN
-F 1 "2.2u" V 2339 1150 50  0000 C CNN
+F 1 "2.2u 10v" V 2339 1150 50  0000 C CNN
 F 2 "Capacitor_SMD:C_0603_1608Metric" H 2538 1000 50  0001 C CNN
 F 3 "~" H 2500 1150 50  0001 C CNN
+F 4 "C167329" V 2500 1150 50  0001 C CNN "LCSC"
 	1    2500 1150
 	0    1    1    0
@@
 P 3325 1725
 F 0 "C4" H 3440 1771 50  0000 L CNN
-F 1 "2.2u" H 3440 1680 50  0000 L CNN
+F 1 "2.2u 10v" H 3440 1680 50  0000 L CNN
 F 2 "Capacitor_SMD:C_0603_1608Metric" H 3363 1575 50  0001 C CNN
 F 3 "~" H 3325 1725 50  0001 C CNN
+F 4 "C167329" H 3325 1725 50  0001 C CNN "LCSC"
 	1    3325 1725
 	1    0    0    -1
@@
 P 4200 1725
 F 0 "C5" H 4315 1771 50  0000 L CNN
-F 1 "10u" H 4315 1680 50  0000 L CNN
+F 1 "10u 10v" H 4315 1680 50  0000 L CNN
 F 2 "Capacitor_SMD:C_0603_1608Metric" H 4238 1575 50  0001 C CNN
 F 3 "~" H 4200 1725 50  0001 C CNN
+F 4 "C195004" H 4200 1725 50  0001 C CNN "LCSC"
 	1    4200 1725
 	1    0    0    -1
@@
 P 3125 1650
 F 0 "C2" H 3025 1725 50  0000 L CNN
-F 1 "10u" H 3050 1575 50  0000 L CNN
+F 1 "10u 10v" H 3050 1575 50  0000 L CNN
 F 2 "Capacitor_SMD:C_0603_1608Metric" H 3163 1500 50  0001 C CNN
 F 3 "~" H 3125 1650 50  0001 C CNN
+F 4 "C195004" H 3125 1650 50  0001 C CNN "LCSC"
 	1    3125 1650
 	1    0    0    -1
@@
 P 3125 2550
 F 0 "C3" H 3240 2596 50  0000 L CNN
-F 1 "2.2u" H 3240 2505 50  0000 L CNN
+F 1 "2.2u 10v" H 3240 2505 50  0000 L CNN
 F 2 "Capacitor_SMD:C_0603_1608Metric" H 3163 2400 50  0001 C CNN
 F 3 "~" H 3125 2550 50  0001 C CNN
+F 4 "C167329" H 3125 2550 50  0001 C CNN "LCSC"
 	1    3125 2550
 	1    0    0    -1
@@
 P 8200 4350
 F 0 "Q1" H 8406 4304 50  0000 L CNN
-F 1 "NDS3332P" H 8406 4395 50  0000 L CNN
+F 1 "NDS332P" H 8406 4395 50  0000 L CNN
 F 2 "Package_TO_SOT_SMD:SOT-23" H 8400 4275 50  0001 L CIN
 F 3 "http://www.onsemi.com/pub/Collateral/NTR2101P-D.PDF" H 8200 4350 50  0001 L CNN
+F 4 "C258217" H 8200 4350 50  0001 C CNN "LCSC"
 	1    8200 4350
 	1    0    0    1
@@
 P 8225 5425
 F 0 "Q2" H 8431 5379 50  0000 L CNN
-F 1 "NDS3332P" H 8431 5470 50  0000 L CNN
+F 1 "NDS332P" H 8431 5470 50  0000 L CNN
 F 2 "Package_TO_SOT_SMD:SOT-23" H 8425 5350 50  0001 L CIN
 F 3 "http://www.onsemi.com/pub/Collateral/NTR2101P-D.PDF" H 8225 5425 50  0001 L CNN
+F 4 "C258217" H 8225 5425 50  0001 C CNN "LCSC"
 	1    8225 5425
 	1    0    0    1
@@
 P 8250 1450
 F 0 "Q3" H 8456 1404 50  0000 L CNN
-F 1 "NDS3332P" H 8456 1495 50  0000 L CNN
+F 1 "NDS332P" H 8456 1495 50  0000 L CNN
 F 2 "Package_TO_SOT_SMD:SOT-23" H 8450 1375 50  0001 L CIN
 F 3 "http://www.onsemi.com/pub/Collateral/NTR2101P-D.PDF" H 8250 1450 50  0001 L CNN
+F 4 "C258217" H 8250 1450 50  0001 C CNN "LCSC"
 	1    8250 1450
 	1    0    0    1
@@
 F 2 "Resistor_SMD:R_0603_1608Metric" V 7880 4175 50  0001 C CNN
 F 3 "~" H 7950 4175 50  0001 C CNN
+F 4 "C191318" H 7950 4175 50  0001 C CNN "LCSC"
 	1    7950 4175
 	1    0    0    -1
@@
 F 2 "Resistor_SMD:R_0603_1608Metric" V 7880 5200 50  0001 C CNN
 F 3 "~" H 7950 5200 50  0001 C CNN
+F 4 "C191318" H 7950 5200 50  0001 C CNN "LCSC"
 	1    7950 5200
 	1    0    0    -1
@@
 F 2 "Resistor_SMD:R_0603_1608Metric" V 7905 1225 50  0001 C CNN
 F 3 "~" H 7975 1225 50  0001 C CNN
+F 4 "C191318" H 7975 1225 50  0001 C CNN "LCSC"
 	1    7975 1225
 	1    0    0    -1
@@
 P 1225 2325
 F 0 "R5" V 1150 2200 50  0000 C CNN
-F 1 "R" V 1475 2275 50  0000 C CNN
+F 1 "1.18k" V 1150 2475 50  0000 C CNN
 F 2 "Resistor_SMD:R_0603_1608Metric" V 1155 2325 50  0001 C CNN
 F 3 "~" H 1225 2325 50  0001 C CNN
+F 4 "C402894" V 1225 2325 50  0001 C CNN "LCSC"
 	1    1225 2325
 	0    1    1    0
@@
 P 1225 2425
 F 0 "R6" V 1300 2275 50  0000 C CNN
-F 1 "R" V 1025 2550 50  0000 C CNN
+F 1 "1.13k" V 1300 2575 50  0000 C CNN
 F 2 "Resistor_SMD:R_0603_1608Metric" V 1155 2425 50  0001 C CNN
 F 3 "~" H 1225 2425 50  0001 C CNN
+F 4 "C308182" V 1225 2425 50  0001 C CNN "LCSC"
 	1    1225 2425
 	0    1    1    0
@@
 F 2 "Package_SO:SOIC-8_3.9x4.9mm_P1.27mm" H 5325 3875 50  0001 C CNN
 F 3 "http://www.wch.cn/downloads/file/240.html" H 5375 3325 50  0001 C CNN
+F 4 "C108996" H 5475 3125 50  0001 C CNN "LCSC"
 	1    5475 3125
 	1    0    0    -1
@@
 Text Label 1400 2125 0    50   ~ 0
 +5V
-$Comp
-L Power_Supervisor:TPS3831 U6
-U 1 1 5E67ED9A
-P 1825 4850
-F 0 "U6" H 2269 4896 50  0000 L CNN
-F 1 "TPS3831" H 2269 4805 50  0000 L CNN
-F 2 "Package_SON:Texas_X2SON-4_1x1mm_P0.65mm" H 1825 4250 50  0001 C CNN
-F 3 "http://www.ti.com/lit/ds/sbvs193d/sbvs193d.pdf" H 1825 4850 50  0001 C CNN
-	1    1825 4850
-	1    0    0    -1
-$EndComp
 Wire Wire Line
 	2225 4850 3100 4850
@@
 Wire Wire Line
 	1825 5350 1875 5350
-Wire Wire Line
-	1925 5350 1925 5150
 $Comp
 L power:GND #PWR013
@@
 Wire Wire Line
 	3700 4325 3700 4225
-Wire Wire Line
-	1525 4850 975  4850
-Text Label 1050 4850 0    50   ~ 0
-~RESET
 Wire Wire Line
 	1275 4250 1275 4500
@@
 F 2 "Resistor_SMD:R_0603_1608Metric" V 2780 2725 50  0001 C CNN
 F 3 "~" H 2850 2725 50  0001 C CNN
+F 4 "C191318" H 2850 2725 50  0001 C CNN "LCSC"
 	1    2850 2725
 	1    0    0    -1
@@
 F 2 "Resistor_SMD:R_0603_1608Metric" V 7230 1650 50  0001 C CNN
 F 3 "~" H 7300 1650 50  0001 C CNN
+F 4 "C427267" V 7300 1650 50  0001 C CNN "LCSC"
 	1    7300 1650
 	0    1    1    0
@@
 F 2 "Package_TO_SOT_SMD:SOT-23" H 7975 1575 50  0001 L CIN
 F 3 "http://www.fairchildsemi.com/ds/PN/PN2222A.pdf" H 7775 1650 50  0001 L CNN
+F 4 "C151009" H 7775 1650 50  0001 C CNN "LCSC"
 	1    7775 1650
 	1    0    0    -1
@@
 F 2 "Resistor_SMD:R_0603_1608Metric" V 7455 1850 50  0001 C CNN
 F 3 "~" H 7525 1850 50  0001 C CNN
+F 4 "C191318" H 7525 1850 50  0001 C CNN "LCSC"
 	1    7525 1850
 	1    0    0    -1
@@
 F 2 "Package_TO_SOT_SMD:SOT-363_SC-70-6" H 7850 4650 50  0001 C CNN
 F 3 "http://www.diodes.com/_files/datasheets/ds30125.pdf" H 7650 4550 50  0001 C CNN
+F 4 "C96379" H 7650 4550 50  0001 C CNN "LCSC"
 	1    7650 4550
 	1    0    0    -1
@@
 F 2 "Package_TO_SOT_SMD:SOT-363_SC-70-6" H 7775 5725 50  0001 C CNN
 F 3 "http://www.diodes.com/_files/datasheets/ds30125.pdf" H 7575 5625 50  0001 C CNN
+F 4 "C96379" H 7575 5625 50  0001 C CNN "LCSC"
 	2    7575 5625
 	1    0    0    -1
@@
 F 2 "Resistor_SMD:R_0603_1608Metric" V 7105 5775 50  0001 C CNN
 F 3 "~" H 7175 5775 50  0001 C CNN
+F 4 "C191318" H 7175 5775 50  0001 C CNN "LCSC"
 	1    7175 5775
 	1    0    0    -1
@@
 F 2 "Resistor_SMD:R_0603_1608Metric" V 7105 4700 50  0001 C CNN
 F 3 "~" H 7175 4700 50  0001 C CNN
+F 4 "C191318" H 7175 4700 50  0001 C CNN "LCSC"
 	1    7175 4700
 	1    0    0    -1
@@
 F 2 "Resistor_SMD:R_0603_1608Metric" V 6880 4525 50  0001 C CNN
 F 3 "~" H 6950 4525 50  0001 C CNN
+F 4 "C427267" V 6950 4525 50  0001 C CNN "LCSC"
 	1    6950 4525
 	0    1    1    0
@@
 F 2 "Resistor_SMD:R_0603_1608Metric" V 6855 5600 50  0001 C CNN
 F 3 "~" H 6925 5600 50  0001 C CNN
+F 4 "C427267" V 6925 5600 50  0001 C CNN "LCSC"
 	1    6925 5600
 	0    1    1    0
@@
 Wire Wire Line
 	7525 6000 7525 5975
+Connection ~ 7525 5975
+Wire Wire Line
+	7525 5975 7175 5975
+$Comp
+L Power_Supervisor:TPS3839DBZ U6
+U 1 1 5EA79CCF
+P 1825 4850
+F 0 "U6" H 1695 4896 50  0000 R CNN
+F 1 "TPS3839DBZ" H 1695 4805 50  0000 R CNN
+F 2 "Package_TO_SOT_SMD:SOT-23" H 1825 4850 50  0001 C CNN
+F 3 "http://www.ti.com/lit/ds/sbvs193d/sbvs193d.pdf" H 1825 4850 50  0001 C CNN
+F 4 "C96333" H 1825 4850 50  0001 C CNN "LCSC"
+	1    1825 4850
+	1    0    0    -1
+$EndComp
 Wire Bus Line
 	2750 5875 2750 6825
-Connection ~ 7525 5975
-Wire Wire Line
-	7525 5975 7175 5975
 $EndSCHEMATC

Commit message: position file
Parts:
- J3: footprint Connector_Card:microSD_HC_Wuerth_693072010801 -> Connector_Card:microSD_HC_Hirose_DM3D-SF
Changed lines of the file:
@@
 F 0 "J3" H 1500 5583 50  0000 C CNN
 F 1 "Micro_SD_Card" H 1500 5674 50  0000 C CNN
-F 2 "Connector_Card:microSD_HC_Wuerth_693072010801" H 2700 6700 50  0001 C CNN
+F 2 "Connector_Card:microSD_HC_Hirose_DM3D-SF" H 2700 6700 50  0001 C CNN
 F 3 "http://katalog.we-online.de/em/datasheet/693072010801.pdf" H 1550 6400 50  0001 C CNN
 	1    1550 6400

Commit message: create files for ordering
Parts:
- J4: LCSC (none) -> C46391
Changed lines of the file:
@@
 F 2 "Connector_USB:USB_Mini-B_Lumberg_2486_01_Horizontal" H 4550 3150 50  0001 C CNN
 F 3 "~" H 4550 3150 50  0001 C CNN
+F 4 "C46391" H 4400 3200 50  0001 C CNN "LCSC"
 	1    4400 3200
 	1    0    0    -1

Commit message: update parts to use all 0603, move labels to be legible
Parts:
- C1, C3, C4: LCSC C167329 -> C23630
- C2, C5: LCSC C195004 -> C19702
- R1, R11, R2: LCSC C427267 -> C22962
- R10, R12, R3, R4, R7, R8, R9: LCSC C191318 -> C25804
- U5: LCSC C126019 -> C23984
Changed lines of the file:
@@
 F 2 "Package_TO_SOT_SMD:SOT-223-3_TabPin2" H 3800 1575 50  0001 C CNN
 F 3 "http://www.ti.com/lit/ds/symlink/lm1117.pdf" H 3800 1575 50  0001 C CNN
-F 4 "C126019" H 3800 1575 50  0001 C CNN "LCSC"
+F 4 "C23984" H 3800 1575 50  0001 C CNN "LCSC"
 	1    3800 1575
 	1    0    0    -1
@@
 F 2 "Capacitor_SMD:C_0603_1608Metric" H 2538 1000 50  0001 C CNN
 F 3 "~" H 2500 1150 50  0001 C CNN
-F 4 "C167329" V 2500 1150 50  0001 C CNN "LCSC"
+F 4 "C23630" V 2500 1150 50  0001 C CNN "LCSC"
 	1    2500 1150
 	0    1    1    0
@@
 F 2 "Capacitor_SMD:C_0603_1608Metric" H 3363 1575 50  0001 C CNN
 F 3 "~" H 3325 1725 50  0001 C CNN
-F 4 "C167329" H 3325 1725 50  0001 C CNN "LCSC"
+F 4 "C23630" H 3325 1725 50  0001 C CNN "LCSC"
 	1    3325 1725
 	1    0    0    -1
@@
 F 2 "Capacitor_SMD:C_0603_1608Metric" H 4238 1575 50  0001 C CNN
 F 3 "~" H 4200 1725 50  0001 C CNN
-F 4 "C195004" H 4200 1725 50  0001 C CNN "LCSC"
+F 4 "C19702" H 4200 1725 50  0001 C CNN "LCSC"
 	1    4200 1725
 	1    0    0    -1
@@
 F 2 "Capacitor_SMD:C_0603_1608Metric" H 3163 1500 50  0001 C CNN
 F 3 "~" H 3125 1650 50  0001 C CNN
-F 4 "C195004" H 3125 1650 50  0001 C CNN "LCSC"
+F 4 "C19702" H 3125 1650 50  0001 C CNN "LCSC"
 	1    3125 1650
 	1    0    0    -1
@@
 F 2 "Capacitor_SMD:C_0603_1608Metric" H 3163 2400 50  0001 C CNN
 F 3 "~" H 3125 2550 50  0001 C CNN
-F 4 "C167329" H 3125 2550 50  0001 C CNN "LCSC"
+F 4 "C23630" H 3125 2550 50  0001 C CNN "LCSC"
 	1    3125 2550
 	1    0    0    -1
@@
 F 2 "Resistor_SMD:R_0603_1608Metric" V 7880 4175 50  0001 C CNN
 F 3 "~" H 7950 4175 50  0001 C CNN
-F 4 "C191318" H 7950 4175 50  0001 C CNN "LCSC"
+F 4 "C25804" H 7950 4175 50  0001 C CNN "LCSC"
 	1    7950 4175
 	1    0    0    -1
@@
 F 2 "Resistor_SMD:R_0603_1608Metric" V 7880 5200 50  0001 C CNN
 F 3 "~" H 7950 5200 50  0001 C CNN
-F 4 "C191318" H 7950 5200 50  0001 C CNN "LCSC"
+F 4 "C25804" H 7950 5200 50  0001 C CNN "LCSC"
 	1    7950 5200
 	1    0    0    -1
@@
 F 2 "Resistor_SMD:R_0603_1608Metric" V 7905 1225 50  0001 C CNN
 F 3 "~" H 7975 1225 50  0001 C CNN
-F 4 "C191318" H 7975 1225 50  0001 C CNN "LCSC"
+F 4 "C25804" H 7975 1225 50  0001 C CNN "LCSC"
 	1    7975 1225
 	1    0    0    -1
@@
 F 2 "Resistor_SMD:R_0603_1608Metric" V 2780 2725 50  0001 C CNN
 F 3 "~" H 2850 2725 50  0001 C CNN
-F 4 "C191318" H 2850 2725 50  0001 C CNN "LCSC"
+F 4 "C25804" H 2850 2725 50  0001 C CNN "LCSC"
 	1    2850 2725
 	1    0    0    -1
@@
 F 2 "Resistor_SMD:R_0603_1608Metric" V 7230 1650 50  0001 C CNN
 F 3 "~" H 7300 1650 50  0001 C CNN
-F 4 "C427267" V 7300 1650 50  0001 C CNN "LCSC"
+F 4 "C22962" V 7300 1650 50  0001 C CNN "LCSC"
 	1    7300 1650
 	0    1    1    0
@@
 F 2 "Resistor_SMD:R_0603_1608Metric" V 7455 1850 50  0001 C CNN
 F 3 "~" H 7525 1850 50  0001 C CNN
-F 4 "C191318" H 7525 1850 50  0001 C CNN "LCSC"
+F 4 "C25804" H 7525 1850 50  0001 C CNN "LCSC"
 	1    7525 1850
 	1    0    0    -1
@@
 F 2 "Resistor_SMD:R_0603_1608Metric" V 7105 5775 50  0001 C CNN
 F 3 "~" H 7175 5775 50  0001 C CNN
-F 4 "C191318" H 7175 5775 50  0001 C CNN "LCSC"
+F 4 "C25804" H 7175 5775 50  0001 C CNN "LCSC"
 	1    7175 5775
 	1    0    0    -1
@@
 F 2 "Resistor_SMD:R_0603_1608Metric" V 7105 4700 50  0001 C CNN
 F 3 "~" H 7175 4700 50  0001 C CNN
-F 4 "C191318" H 7175 4700 50  0001 C CNN "LCSC"
+F 4 "C25804" H 7175 4700 50  0001 C CNN "LCSC"
 	1    7175 4700
 	1    0    0    -1
@@
 F 2 "Resistor_SMD:R_0603_1608Metric" V 6880 4525 50  0001 C CNN
 F 3 "~" H 6950 4525 50  0001 C CNN
-F 4 "C427267" V 6950 4525 50  0001 C CNN "LCSC"
+F 4 "C22962" V 6950 4525 50  0001 C CNN "LCSC"
 	1    6950 4525
 	0    1    1    0
@@
 F 2 "Resistor_SMD:R_0603_1608Metric" V 6855 5600 50  0001 C CNN
 F 3 "~" H 6925 5600 50  0001 C CNN
-F 4 "C427267" V 6925 5600 50  0001 C CNN "LCSC"
+F 4 "C22962" V 6925 5600 50  0001 C CNN "LCSC"
 	1    6925 5600
 	0    1    1    0
